File: hardware/psu_lm2576.kicad_sch (KiCad schematic)
At the start: 6 parts, among them U16 LM2576S-5_0_TR, U17 100uH

Commit message: replace 1000uF capacitor with in stock part
Parts:
- C28: LCSC C310843 -> C280408
Changed lines of the file:
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@@
 			)
 		)
-		(property "LCSC" "C310843"
+		(property "LCSC" "C280408"
 			(at 173.99 99.06 0)
 			(effects
